File: led-planets.kicad_sch (KiCad schematic)
At the start: 0 parts

Commit message: starting schematic
Parts:
- added U1: ARDUINO_PRO_MINI, jannett_footprints:MODULE_ARDUINO_PRO_MINI, symbol jannett_symbols:ARDUINO_PRO_MINI
Connections:
- new net: U1.JP1_5 (GND), U1.JP1_6 (GND)
Changed lines of the file:
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@@
 	(generator_version "9.0")
 	(paper "A4")
+	(symbol
+		(lib_id "jannett_symbols:ARDUINO_PRO_MINI")
+		(at 69.85 69.85 0)
+		(unit 1)
+		(exclude_from_sim no)
+		(in_bom yes)
+		(on_board yes)
+		(dnp no)
+		(fields_autoplaced yes)
+		(property "Reference" "U1"
+			(at 69.85 34.29 0)
+			(effects
+				(font
+					(size 1.27 1.27)
+				)
+			)
+		)
+		(property "Value" "ARDUINO_PRO_MINI"
+			(at 69.85 36.83 0)
+			(effects
+				(font
+					(size 1.27 1.27)
+				)
+			)
+		)
+		(property "Footprint" "jannett_footprints:MODULE_ARDUINO_PRO_MINI"
+			(at 69.85 69.85 0)
+			(effects
+				(font
+					(size 1.27 1.27)
+				)
+				(justify left bottom)
+				(hide yes)
+			)
+		)
+		(property "Datasheet" ""
+			(at 69.85 69.85 0)
+			(effects
+				(font
+					(size 1.27 1.27)
+				)
+				(justify left bottom)
+				(hide yes)
+			)
+		)
+		(property "Description" ""
+			(at 69.85 69.85 0)
+			(effects
+				(font
+					(size 1.27 1.27)
+				)
+				(hide yes)
+			)
+		)
+		(property "MAXIMUM_PACKAGE_HEIGHT" "N/A"
+			(at 69.85 69.85 0)
+			(effects
+				(font
+					(size 1.27 1.27)
+				)
+				(justify left bottom)
+				(hide yes)
+			)
+		)
+		(property "STANDARD" "Manufacturer Recommendations"
+			(at 69.85 69.85 0)
+			(effects
+				(font
+					(size 1.27 1.27)
+				)
+				(justify left bottom)
+				(hide yes)
+			)
+		)
+		(property "PARTREV" "N/A"
+			(at 69.85 69.85 0)
+			(effects
+				(font
+					(size 1.27 1.27)
+				)
+				(justify left bottom)
+				(hide yes)
+			)
+		)
+		(property "MANUFACTURER" "SparkFun Electronics"
+			(at 69.85 69.85 0)
+			(effects
+				(font
+					(size 1.27 1.27)
+				)
+				(justify left bottom)
+				(hide yes)
+			)
+		)
+		(pin "JP2_1"
+		)
+		(pin "JP3_1"
+		)
+		(pin "JP3_2"
+		)
+		(pin "JP7_12"
+		)
+		(pin "JP7_8"
+		)
+		(pin "JP6_12"
+		)
+		(pin "JP6_8"
+		)
+		(pin "JP6_11"
+		)
+		(pin "JP6_1"
+		)
+		(pin "JP1_3"
+		)
+		(pin "JP7_10"
+		)
+		(pin "JP7_3"
+		)
+		(pin "JP6_6"
+		)
+		(pin "JP1_4"
+		)
+		(pin "JP6_5"
+		)
+		(pin "JP6_7"
+		)
+		(pin "JP6_3"
+		)
+		(pin "JP6_10"
+		)
+		(pin "JP1_1"
+		)
+		(pin "JP6_4"
+		)
+		(pin "JP1_2"
+		)
+		(pin "JP2_2"
+		)
+		(pin "JP6_9"
+		)
+		(pin "JP7_11"
+		)
+		(pin "JP7_7"
+		)
+		(pin "JP7_6"
+		)
+		(pin "JP7_5"
+		)
+		(pin "JP7_4"
+		)
+		(pin "JP7_2"
+		)
+		(pin "JP7_1"
+		)
+		(pin "JP1_5"
+		)
+		(pin "JP7_9"
+		)
+		(pin "JP6_2"
+		)
+		(pin "JP1_6"
+		)
+		(instances
+			(project ""
+				(path "/8ea47bf3-e487-4b21-a6f2-a91dd50001f4"
+					(reference "U1")
+					(unit 1)
+				)
+			)
+		)
+	)
 	(sheet_instances
 		(path "/"

Commit message: schematic changes
Parts:
- added C1, C2, C3, C4, C5, C6, C7, C8, C9: 22uF, Capacitor_SMD:C_0603_1608Metric_Pad1.08x0.95mm_HandSolder, symbol Device:C_Small
- added J1, J2: SM08B-GHS-TB, Connector_JST:JST_GH_SM08B-GHS-TB_1x08-1MP_P1.25mm_Horizontal, symbol Connector_Generic:Conn_01x08
- added J3: USB4135-GF-A, Connector_USB:USB_C_Receptacle_GCT_USB4135-GF-A_6P_TopMnt_Horizontal, symbol Connector:USB_C_Receptacle_PowerOnly_6P
- added Q1, Q2, Q3, Q4, Q5, Q6, Q7, Q8: MMBT2222A, Package_TO_SOT_SMD:SOT-23, symbol Transistor_BJT:MMBT2222A
- added R1, R2, R3, R4, R5, R6, R7, R8, R9: 20K, Resistor_SMD:R_0603_1608Metric_Pad0.98x0.95mm_HandSolder, symbol Device:R_US
- added R10: R_Photo, OptoDevice:R_LDR_5.0x4.1mm_P3mm_Vertical, symbol Device:R_Photo
Connections:
- net +5V: now reaches U1.JP1_4 (VCC)
- net +5V: now also U1.JP6_4 (VCC_1), C9.1, J3.A9 (VBUS), J3.B9 (VBUS), R9.2
- net GND: now reaches U1.JP1_5 (GND), U1.JP1_6 (GND)
- net GND: now also U1.JP6_2 (GND_1), U1.JP7_9 (GND_2), C1.2, C2.2, C3.2, C4.2, C5.2, C6.2, C7.2, C8.2, C9.2, J3.A12 (GND), J3.B12 (GND), J3.S1 (SHIELD), Q1.2 (E), Q2.2 (E), Q3.2 (E), Q4.2 (E), Q5.2 (E), Q6.2 (E), Q7.2 (E), Q8.2 (E), R10.2
- net A0: now reaches U1.JP6_8 (A0)
- net A0: now also R10.1, R9.1
- new net: C6.1, Q6.1 (B), R6.2
- new net: C4.1, Q4.1 (B), R4.2
- new net: C2.1, Q2.1 (B), R2.2
- new net: C5.1, Q5.1 (B), R5.2
- new net: C7.1, Q7.1 (B), R7.2
- new net: C1.1, Q1.1 (B), R1.2
- new net: C3.1, Q3.1 (B), R3.2
- new net: C8.1, Q8.1 (B), R8.2

Commit message: layout and sch
Parts:
- added R11, R12, R13, R14, R15, R16, R17, R18: 100, Resistor_SMD:R_0603_1608Metric_Pad0.98x0.95mm_HandSolder, symbol Device:R_US
Connections:
- net +5V: now also J1.1 (Pin_1), J1.3 (Pin_3), J1.5 (Pin_5), J1.7 (Pin_7), J2.1 (Pin_1), J2.3 (Pin_3), J2.5 (Pin_5), J2.7 (Pin_7)
- net at Q6.3 (C): now also R16.1
- net D3: now reaches R2.1
- net D3: now also U1.JP7_7 (D3)
- net D9: now reaches U1.JP7_1 (D9)
- net D9: now also R8.1
- net D8: now reaches U1.JP7_2 (D8)
- net D8: now also R7.1
- net D7: now reaches U1.JP7_3 (D7)
- net D7: now also R6.1
- net D6: now reaches U1.JP7_4 (D6)
- net D6: now also R5.1
- net D5: now reaches U1.JP7_5 (D5)
- net D5: now also R4.1
- net D4: now reaches U1.JP7_6 (D4)
- net D4: now also R3.1
- net D2: now reaches U1.JP7_8 (D2)
- net D2: now also R1.1
- net MER: now reaches J1.2 (Pin_2)
- net MER: now also R11.2
- net VEN: now reaches J1.4 (Pin_4)
- net VEN: now also R12.2
- net EAR: now reaches J1.6 (Pin_6)
- net EAR: now also R13.2
- net MAR: now reaches J1.8 (Pin_8)
- net MAR: now also R14.2
- net at Q7.3 (C): now also R17.1
- net at Q1.3 (C): now also R11.1
- net at Q2.3 (C): now also R12.1
- net JUP: now reaches J2.2 (Pin_2)
- net JUP: now also R15.2
- net SAT: now reaches J2.4 (Pin_4)
- net SAT: now also R16.2
- net URA: now reaches J2.6 (Pin_6)
- net URA: now also R17.2
- net NEP: now reaches J2.8 (Pin_8)
- net NEP: now also R18.2
- net at Q5.3 (C): now also R15.1
- net at Q3.3 (C): now also R13.1
- net at Q4.3 (C): now also R14.1
- net at Q8.3 (C): now also R18.1

Commit message: schematic
Parts:
- removed U1: ARDUINO_PRO_MINI, jannett_footprints:MODULE_ARDUINO_PRO_MINI, symbol jannett_symbols:ARDUINO_PRO_MINI
- added U2: ESP32 Module, jannett_footprints:ESP32_MODULE, symbol jannett_symbols:ESP32_Module
Changed lines of the file:
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@@
-	)
-	(symbol
-		(lib_id "jannett_symbols:ARDUINO_PRO_MINI")
-		(at 69.85 69.85 0)
-		(unit 1)
-		(exclude_from_sim no)
-		(in_bom yes)
-		(on_board yes)
-		(dnp no)
-		(fields_autoplaced yes)
-		(property "Reference" "U1"
-			(at 69.85 34.29 0)
-			(effects
-				(font
-					(size 1.27 1.27)
-				)
-			)
-		)
-		(property "Value" "ARDUINO_PRO_MINI"
-			(at 69.85 36.83 0)
-			(effects
-				(font
-					(size 1.27 1.27)
-				)
-			)
-		)
-		(property "Footprint" "jannett_footprints:MODULE_ARDUINO_PRO_MINI"
-			(at 69.85 69.85 0)
-			(effects
-				(font
-					(size 1.27 1.27)
-				)
-				(justify left bottom)
-				(hide yes)
-			)
-		)
-		(property "Datasheet" ""
-			(at 69.85 69.85 0)
-			(effects
-				(font
-					(size 1.27 1.27)
-				)
-				(justify left bottom)
-				(hide yes)
-			)
-		)
-		(property "Description" ""
-			(at 69.85 69.85 0)
-			(effects
-				(font
-					(size 1.27 1.27)
-				)
-				(hide yes)
-			)
-		)
-		(property "MAXIMUM_PACKAGE_HEIGHT" "N/A"
-			(at 69.85 69.85 0)
-			(effects
-				(font
-					(size 1.27 1.27)
-				)
-				(justify left bottom)
-				(hide yes)
-			)
-		)
-		(property "STANDARD" "Manufacturer Recommendations"
-			(at 69.85 69.85 0)
-			(effects
-				(font
-					(size 1.27 1.27)
-				)
-				(justify left bottom)
-				(hide yes)
-			)
-		)
-		(property "PARTREV" "N/A"
-			(at 69.85 69.85 0)
-			(effects
-				(font
-					(size 1.27 1.27)
-				)
-				(justify left bottom)
-				(hide yes)
-			)
-		)
-		(property "MANUFACTURER" "SparkFun Electronics"
-			(at 69.85 69.85 0)
-			(effects
-				(font
-					(size 1.27 1.27)
-				)
-				(justify left bottom)
-				(hide yes)
-			)
-		)
-		(pin "JP2_1"
-		)
-		(pin "JP3_1"
-		)
-		(pin "JP3_2"
-		)
-		(pin "JP7_12"
-		)
-		(pin "JP7_8"
-		)
-		(pin "JP6_12"
-		)
-		(pin "JP6_8"
-		)
-		(pin "JP6_11"
-		)
-		(pin "JP6_1"
-		)
-		(pin "JP1_3"
-		)
-		(pin "JP7_10"
-		)
-		(pin "JP7_3"
-		)
-		(pin "JP6_6"
-		)
-		(pin "JP1_4"
-		)
-		(pin "JP6_5"
-		)
-		(pin "JP6_7"
-		)
-		(pin "JP6_3"
-		)
-		(pin "JP6_10"
-		)
-		(pin "JP1_1"
-		)
-		(pin "JP6_4"
-		)
-		(pin "JP1_2"
-		)
-		(pin "JP2_2"
-		)
-		(pin "JP6_9"
-		)
-		(pin "JP7_11"
-		)
-		(pin "JP7_7"
-		)
-		(pin "JP7_6"
-		)
-		(pin "JP7_5"
-		)
-		(pin "JP7_4"
-		)
-		(pin "JP7_2"
-		)
-		(pin "JP7_1"
-		)
-		(pin "JP1_5"
-		)
-		(pin "JP7_9"
-		)
-		(pin "JP6_2"
-		)
-		(pin "JP1_6"
-		)
-		(instances
-			(project ""
-				(path "/8ea47bf3-e487-4b21-a6f2-a91dd50001f4"
-					(reference "U1")
-					(unit 1)
-				)
-			)
-		)
 	)
 	(symbol
@@
 					(unit 1)
 				)
+			)
+		)
+	)
+	(symbol
+		(lib_id "jannett_symbols:ESP32_Module")
+		(at 142.24 146.05 0)
+		(unit 1)
+		(exclude_from_sim no)
+		(in_bom yes)
+		(on_board yes)
+		(dnp no)
+		(fields_autoplaced yes)
+		(property "Reference" "U2"
+			(at 151.13 142.24 0)
+			(effects
+				(font
+					(size 1.27 1.27)
+				)
+			)
+		)
+		(property "Value" "ESP32 Module"
+			(at 151.13 144.78 0)
+			(effects
+				(font
+					(size 1.27 1.27)
+				)
+			)
+		)
+		(property "Footprint" "jannett_footprints:ESP32_MODULE"
+			(at 142.24 146.05 0)
+			(effects
+				(font
+					(size 1.27 1.27)
+				)
+				(hide yes)
+			)
+		)
+		(property "Datasheet" ""
+			(at 142.24 146.05 0)
+			(effects
+				(font
+					(size 1.27 1.27)
+				)
+				(hide yes)
+			)
+		)
+		(property "Description" ""
+			(at 142.24 146.05 0)
+			(effects
+				(font
+					(size 1.27 1.27)
+				)
+				(hide yes)
+			)
+		)
+		(pin "4"
+		)
+		(pin "29"
+		)
+		(pin "26"
+		)
+		(pin "23"
+		)
+		(pin "21"
+		)
+		(pin "12"
+		)
+		(pin "9"
+		)
+		(pin "30"
+		)
+		(pin "1"
+		)
+		(pin "2"
+		)
+		(pin "5"
+		)
+		(pin "7"
+		)
+		(pin "28"
+		)
+		(pin "8"
+		)
+		(pin "10"
+		)
+		(pin "11"
+		)
+		(pin "13"
+		)
+		(pin "15"
+		)
+		(pin "3"
+		)
+		(pin "14"
+		)
+		(pin "6"
+		)
+		(pin "27"
+		)
+		(pin "25"
+		)
+		(pin "24"
+		)
+		(pin "22"
+		)
+		(pin "16"
+		)
+		(pin "19"
+		)
+		(pin "20"
+		)
+		(pin "17"
+		)
+		(pin "18"
+		)
+		(instances
+			(project ""
+				(path "/8ea47bf3-e487-4b21-a6f2-a91dd50001f4"
+					(reference "U2")
+					(unit 1)
+				)

Commit message: schematic finished
Parts:
- removed J3: USB4135-GF-A, Connector_USB:USB_C_Receptacle_GCT_USB4135-GF-A_6P_TopMnt_Horizontal, symbol Connector:USB_C_Receptacle_PowerOnly_6P
- added C10: 0.1uF, Capacitor_SMD:C_0603_1608Metric_Pad1.08x0.95mm_HandSolder, symbol Device:C_Small
- added J3: Conn_01x05, Connector_PinSocket_2.54mm:PinSocket_1x05_P2.54mm_Vertical, symbol Connector_Generic:Conn_01x05
Connections:
- net A0 is gone; now on net ADC_IN_PHOTO: R10.1, R9.1
- net D2 is gone; now on net MER_B: R1.1
- net D3 is gone; now on net VEN_B: R2.1
- net D4 is gone; now on net EAR_B: R3.1
- net D5 is gone; now on net MAR_B: R4.1
- net D6 is gone; now on net JUP_B: R5.1
- net D7 is gone; now on net SAT_B: R6.1
- net D8 is gone; now on net URA_B: R7.1
- net D9 is gone; now on net NEP_B: R8.1
- net +5V: now also U2.30 (VIN), J3.5 (Pin_5); no longer R9.2
- net GND: now also U2.2 (GND), U2.29 (GND), C10.2, J3.4 (Pin_4)
- net +3.3V: now reaches U2.1 (+3.3V)
- net +3.3V: now also R9.2
- net ADC_IN_PHOTO: now reaches U2.19 (GPIO34)
- net ADC_IN_PHOTO: now also C10.1
- net MER_B: now reaches U2.21 (GPIO32)
- net VEN_B: now reaches U2.22 (GPIO33)
- net EAR_B: now reaches U2.23 (GPIO25)
- net MAR_B: now reaches U2.24 (GPIO26)
- net JUP_B: now reaches U2.25 (GPIO27)
- net SAT_B: now reaches U2.26 (GPIO14)
- net URA_B: now reaches U2.27 (GPIO12)
- net NEP_B: now reaches U2.28 (GPIO13)
- net TX: now reaches U2.6 (GPIO16)
- net TX: now also J3.1 (Pin_1)
- net RX: now reaches U2.7 (GPIO17)
- net RX: now also J3.2 (Pin_2)
- net OUT: now reaches U2.8 (GPIO5)
- net OUT: now also J3.3 (Pin_3)
Other:
- moved on the sheet: C9, R10, R9, U2

Commit message: layout
Parts:
- added H1, H2, H3, H4: M3, MountingHole:MountingHole_3.2mm_M3, symbol Mechanical:MountingHole
- added TP1, TP2, TP3: 5016, jannett_footprints:TestPoint_Keystone_5016_Compact, symbol Connector:TestPoint
Connections:
- net +3.3V: now also TP1.1
- net +5V: now also TP2.1
- net GND: now also TP3.1
