File: led-planets.kicad_pcb (KiCad board)
At the start: 2 copper layers, 2 parts, among them U1 ARDUINO_PRO_MINI, U2 ULN2003ADYY

Commit message: schematic changes
Parts:
- removed U2: ULN2003ADYY, Package_SO:Texas_DYY0016A_TSOT-23-16_2x4.2mm_P0.5mm
- added C1: 22uF, Capacitor_SMD:C_0603_1608Metric_Pad1.08x0.95mm_HandSolder, F.Cu at (123.9, 74.0)
- added C2: 22uF, Capacitor_SMD:C_0603_1608Metric_Pad1.08x0.95mm_HandSolder, F.Cu at (123.9, 76.5)
- added C3: 22uF, Capacitor_SMD:C_0603_1608Metric_Pad1.08x0.95mm_HandSolder, F.Cu at (123.9, 79.0)
- added C4: 22uF, Capacitor_SMD:C_0603_1608Metric_Pad1.08x0.95mm_HandSolder, F.Cu at (123.9, 81.6)
- added C5: 22uF, Capacitor_SMD:C_0603_1608Metric_Pad1.08x0.95mm_HandSolder, F.Cu at (123.9, 84.1)
- added C6: 22uF, Capacitor_SMD:C_0603_1608Metric_Pad1.08x0.95mm_HandSolder, F.Cu at (123.9, 86.6)
- added C7: 22uF, Capacitor_SMD:C_0603_1608Metric_Pad1.08x0.95mm_HandSolder, F.Cu at (123.9, 89.1)
- added C8: 22uF, Capacitor_SMD:C_0603_1608Metric_Pad1.08x0.95mm_HandSolder, F.Cu at (128.2, 74.0)
- added C9: 22uF, Capacitor_SMD:C_0603_1608Metric_Pad1.08x0.95mm_HandSolder, F.Cu at (128.2, 76.5)
- added J1: SM08B-GHS-TB, Connector_JST:JST_GH_SM08B-GHS-TB_1x08-1MP_P1.25mm_Horizontal, F.Cu at (142.5, 76.5)
- added J2: SM08B-GHS-TB, Connector_JST:JST_GH_SM08B-GHS-TB_1x08-1MP_P1.25mm_Horizontal, F.Cu at (142.5, 84.0)
- added J3: USB4135-GF-A, Connector_USB:USB_C_Receptacle_GCT_USB4135-GF-A_6P_TopMnt_Horizontal, F.Cu at (109.6, 53.6)
- added Q1: MMBT2222A, Package_TO_SOT_SMD:SOT-23, F.Cu at (124.2, 66.1)
- added Q2: MMBT2222A, Package_TO_SOT_SMD:SOT-23, F.Cu at (124.2, 70.5)
- added Q3: MMBT2222A, Package_TO_SOT_SMD:SOT-23, F.Cu at (129.1, 66.1)
- added Q4: MMBT2222A, Package_TO_SOT_SMD:SOT-23, F.Cu at (129.1, 70.5)
- added Q5: MMBT2222A, Package_TO_SOT_SMD:SOT-23, F.Cu at (134.0, 66.1)
- added Q6: MMBT2222A, Package_TO_SOT_SMD:SOT-23, F.Cu at (134.0, 70.5)
- added Q7: MMBT2222A, Package_TO_SOT_SMD:SOT-23, F.Cu at (138.9, 66.1)
- added Q8: MMBT2222A, Package_TO_SOT_SMD:SOT-23, F.Cu at (138.9, 70.5)
- added R1: 20K, Resistor_SMD:R_0603_1608Metric_Pad0.98x0.95mm_HandSolder, F.Cu at (128.2, 79.0)
- added R10: R_Photo, OptoDevice:R_LDR_5.0x4.1mm_P3mm_Vertical, F.Cu at (143.0, 66.7)
- added R2: 20K, Resistor_SMD:R_0603_1608Metric_Pad0.98x0.95mm_HandSolder, F.Cu at (128.2, 81.6)
- added R3: 20K, Resistor_SMD:R_0603_1608Metric_Pad0.98x0.95mm_HandSolder, F.Cu at (128.2, 84.1)
- added R4: 20K, Resistor_SMD:R_0603_1608Metric_Pad0.98x0.95mm_HandSolder, F.Cu at (128.2, 86.6)
- added R5: 20K, Resistor_SMD:R_0603_1608Metric_Pad0.98x0.95mm_HandSolder, F.Cu at (128.2, 89.1)
- added R6: 20K, Resistor_SMD:R_0603_1608Metric_Pad0.98x0.95mm_HandSolder, F.Cu at (132.6, 74.0)
- added R7: 20K, Resistor_SMD:R_0603_1608Metric_Pad0.98x0.95mm_HandSolder, F.Cu at (132.6, 76.5)
- added R8: 20K, Resistor_SMD:R_0603_1608Metric_Pad0.98x0.95mm_HandSolder, F.Cu at (132.6, 79.0)
- added R9: 20K, Resistor_SMD:R_0603_1608Metric_Pad0.98x0.95mm_HandSolder, F.Cu at (132.6, 81.6)
Connections:
- U1 pad JP1_4: unconnected-(U1-VCC-PadJP1_4) -> +5V
- U1 pad JP1_5: Net-(U1-GND-PadJP1_5) -> GND
- U1 pad JP1_6: Net-(U1-GND-PadJP1_5) -> GND
- U1 pad JP6_2: unconnected-(U1-GND_1-PadJP6_2) -> GND
- U1 pad JP6_4: unconnected-(U1-VCC_1-PadJP6_4) -> +5V
- U1 pad JP6_8: unconnected-(U1-A0-PadJP6_8) -> /A0
- U1 pad JP7_9: unconnected-(U1-GND_2-PadJP7_9) -> GND

Commit message: layout and sch
Parts:
- added R11: 100, Resistor_SMD:R_0603_1608Metric_Pad0.98x0.95mm_HandSolder, F.Cu at (154.1, 65.9)
- added R12: 100, Resistor_SMD:R_0603_1608Metric_Pad0.98x0.95mm_HandSolder, F.Cu at (154.1, 68.4)
- added R13: 100, Resistor_SMD:R_0603_1608Metric_Pad0.98x0.95mm_HandSolder, F.Cu at (154.1, 71.0)
- added R14: 100, Resistor_SMD:R_0603_1608Metric_Pad0.98x0.95mm_HandSolder, F.Cu at (154.1, 73.5)
- added R15: 100, Resistor_SMD:R_0603_1608Metric_Pad0.98x0.95mm_HandSolder, F.Cu at (154.1, 76.0)
- added R16: 100, Resistor_SMD:R_0603_1608Metric_Pad0.98x0.95mm_HandSolder, F.Cu at (154.1, 78.5)
- added R17: 100, Resistor_SMD:R_0603_1608Metric_Pad0.98x0.95mm_HandSolder, F.Cu at (154.1, 81.0)
- added R18: 100, Resistor_SMD:R_0603_1608Metric_Pad0.98x0.95mm_HandSolder, F.Cu at (154.1, 83.5)
- moved J1 60.8 mm to (82.2, 69.1), turned to -90 degrees
- moved J2 60.4 mm to (82.2, 85.1), turned to -90 degrees
- moved R10 32.3 mm to (125.0, 93.5)
Connections:
- J1 pad 1: unconnected-(J1-Pin_1-Pad1) -> +5V
- J1 pad 2: unconnected-(J1-Pin_2-Pad2) -> /MER
- J1 pad 3: unconnected-(J1-Pin_3-Pad3) -> +5V
- J1 pad 4: unconnected-(J1-Pin_4-Pad4) -> /VEN
- J1 pad 5: unconnected-(J1-Pin_5-Pad5) -> +5V
- J1 pad 6: unconnected-(J1-Pin_6-Pad6) -> /EAR
- J1 pad 7: unconnected-(J1-Pin_7-Pad7) -> +5V
- J1 pad 8: unconnected-(J1-Pin_8-Pad8) -> /MAR
- J2 pad 1: unconnected-(J2-Pin_1-Pad1) -> +5V
- J2 pad 2: unconnected-(J2-Pin_2-Pad2) -> /JUP
- J2 pad 3: unconnected-(J2-Pin_3-Pad3) -> +5V
- J2 pad 4: unconnected-(J2-Pin_4-Pad4) -> /SAT
- J2 pad 5: unconnected-(J2-Pin_5-Pad5) -> +5V
- J2 pad 6: unconnected-(J2-Pin_6-Pad6) -> /URA
- J2 pad 7: unconnected-(J2-Pin_7-Pad7) -> +5V
- J2 pad 8: unconnected-(J2-Pin_8-Pad8) -> /NEP
- Q1 pad 3: unconnected-(Q1-C-Pad3) -> Net-(Q1-C)
- Q2 pad 3: unconnected-(Q2-C-Pad3) -> Net-(Q2-C)
- Q3 pad 3: unconnected-(Q3-C-Pad3) -> Net-(Q3-C)
- Q4 pad 3: unconnected-(Q4-C-Pad3) -> Net-(Q4-C)
- Q5 pad 3: unconnected-(Q5-C-Pad3) -> Net-(Q5-C)
- Q6 pad 3: unconnected-(Q6-C-Pad3) -> Net-(Q6-C)
- Q7 pad 3: unconnected-(Q7-C-Pad3) -> Net-(Q7-C)
- Q8 pad 3: unconnected-(Q8-C-Pad3) -> Net-(Q8-C)
- R1 pad 1: unconnected-(R1-Pad1) -> /D2
- R2 pad 1: unconnected-(R2-Pad1) -> /D3
- R3 pad 1: unconnected-(R3-Pad1) -> /D4
- R4 pad 1: unconnected-(R4-Pad1) -> /D5
- R5 pad 1: unconnected-(R5-Pad1) -> /D6
- R6 pad 1: unconnected-(R6-Pad1) -> /D7
- R7 pad 1: unconnected-(R7-Pad1) -> /D8
- R8 pad 1: unconnected-(R8-Pad1) -> /D9
- U1 pad JP7_1: unconnected-(U1-D9-PadJP7_1) -> /D9
- U1 pad JP7_2: unconnected-(U1-D8-PadJP7_2) -> /D8
- U1 pad JP7_3: unconnected-(U1-D7-PadJP7_3) -> /D7
- U1 pad JP7_4: unconnected-(U1-D6-PadJP7_4) -> /D6
- U1 pad JP7_5: unconnected-(U1-D5-PadJP7_5) -> /D5
- U1 pad JP7_6: unconnected-(U1-D4-PadJP7_6) -> /D4
- U1 pad JP7_7: unconnected-(U1-D3-PadJP7_7) -> /D3
- U1 pad JP7_8: unconnected-(U1-D2-PadJP7_8) -> /D2

Commit message: schematic finished
Parts:
- removed U1: ARDUINO_PRO_MINI, jannett_footprints:MODULE_ARDUINO_PRO_MINI
- added C10: 0.1uF, Capacitor_SMD:C_0603_1608Metric_Pad1.08x0.95mm_HandSolder, F.Cu at (150.4, 68.4)
- added U2: ESP32 Module, jannett_footprints:ESP32_MODULE, F.Cu at (105.0, 73.5)
- J3: value USB4135-GF-A -> Conn_01x05; footprint Connector_USB:USB_C_Receptacle_GCT_USB4135-GF-A_6P_TopMnt_Horizontal -> Connector_PinSocket_2.54mm:PinSocket_1x05_P2.54mm_Vertical
- moved R11 90.2 mm to (63.9, 65.0)
- moved R12 90.2 mm to (63.9, 67.5)
- moved R13 90.2 mm to (63.9, 70.0)
- moved R14 90.2 mm to (63.9, 72.5)
- moved R15 90.2 mm to (63.9, 75.0)
- moved R16 90.2 mm to (63.9, 77.5)
- moved R17 90.2 mm to (63.9, 80.1)
- moved R18 90.2 mm to (63.9, 82.6)
- moved R10 74.5 mm to (62.5, 53.0)
- moved Q8 69.2 mm to (70.5, 80.9), turned to -90 degrees
- moved Q7 65.6 mm to (75.0, 80.9), turned to -90 degrees
- moved Q6 63.7 mm to (70.5, 76.0), turned to -90 degrees
- moved Q5 59.8 mm to (75.0, 76.0), turned to -90 degrees
- moved Q4 58.6 mm to (70.5, 71.1), turned to -90 degrees
- moved Q3 54.3 mm to (75.0, 71.1), turned to -90 degrees
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Connections:
- net /A0 renamed /ADC_IN_PHOTO
- R1 pad 1: /D2 -> /MER_B
- R2 pad 1: /D3 -> /VEN_B
- R3 pad 1: /D4 -> /EAR_B
- R4 pad 1: /D5 -> /MAR_B
- R5 pad 1: /D6 -> /JUP_B
- R6 pad 1: /D7 -> /SAT_B
- R7 pad 1: /D8 -> /URA_B
- R8 pad 1: /D9 -> /NEP_B
- R9 pad 2: +5V -> +3.3V

Commit message: layout
Parts:
- added H1: M3, MountingHole:MountingHole_3.2mm_M3, F.Cu at (50.0, 52.0)
- added H2: M3, MountingHole:MountingHole_3.2mm_M3, F.Cu at (130.0, 52.0)
- added H3: M3, MountingHole:MountingHole_3.2mm_M3, F.Cu at (50.0, 95.0)
- added H4: M3, MountingHole:MountingHole_3.2mm_M3, F.Cu at (130.0, 95.0)
- added TP1: 5016, jannett_footprints:TestPoint_Keystone_5016_Compact, F.Cu at (124.2, 87.8)
- added TP2: 5016, jannett_footprints:TestPoint_Keystone_5016_Compact, F.Cu at (80.3, 93.5)
- added TP3: 5016, jannett_footprints:TestPoint_Keystone_5016_Compact, F.Cu at (80.3, 88.3)
- moved C10 71.5 mm to (80.0, 56.0)
- moved R9 59.8 mm to (80.0, 53.0)
- moved C8 55.1 mm to (74.0, 84.0), turned to 180 degrees
- moved R6 52.3 mm to (80.5, 79.0), turned to 180 degrees
- moved R7 52.3 mm to (80.5, 81.5), turned to 180 degrees
- moved R8 52.3 mm to (80.5, 84.0), turned to 180 degrees
- moved C7 50.4 mm to (74.0, 81.5), turned to 180 degrees
- moved C6 50.4 mm to (74.0, 79.0), turned to 180 degrees
- moved C5 50.4 mm to (74.0, 76.5), turned to 180 degrees
- moved C4 50.4 mm to (74.0, 74.0), turned to 180 degrees
- moved C3 50.4 mm to (74.0, 71.5), turned to 180 degrees
- moved C2 50.4 mm to (74.0, 69.0), turned to 180 degrees
- moved C1 50.4 mm to (74.0, 66.5), turned to 180 degrees
- moved R1 49.4 mm to (80.4, 66.5), turned to 180 degrees
- moved R5 49.4 mm to (80.5, 76.5), turned to 180 degrees
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Routing:
- net GND: track 0.00 -> 256.0 mm, vias 0 -> 18
- net +5V: track 0.00 -> 139.4 mm
- net +3.3V: track 0.00 -> 68.5 mm
- net /ADC_IN_PHOTO: track 0.00 -> 24.1 mm
- net Net-(Q8-B): track 0.00 -> 16.3 mm
- net Net-(Q7-B): track 0.00 -> 15.9 mm
- net Net-(Q6-B): track 0.00 -> 15.5 mm
- net Net-(Q3-B): track 0.00 -> 15.2 mm
- net Net-(Q1-B): track 0.00 -> 15.1 mm
- net Net-(Q5-B): track 0.00 -> 15.1 mm
- net Net-(Q4-B): track 0.00 -> 15.0 mm
- net Net-(Q2-B): track 0.00 -> 14.8 mm
- net /TX: track 0.00 -> 11.3 mm
- net /RX: track 0.00 -> 11.3 mm
- net /OUT: track 0.00 -> 11.3 mm
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Other:
- board outline added: 88 x 51 mm
- board text added: "3.3V"
- board text added: "5V"
- board text added: "ADC 34"
- board text added: "D12"
- board text added: "D13"
- board text added: "D14"
- board text added: "D25"
- board text added: "D26"
- board text added: "D27"
- board text added: "D32"
- board text added: "D33"
- board text added: "D5"
- board text added: "EAR"
- board text added: "ESP32 Dev Module"
- board text added: "GND"
- board text added: "JUP"
- board text added: "Jannett W"
- board text added: "MAR"
- board text added: "MER"
- board text added: "NEP"
- board text added: "OUT"
- board text added: "RX"
- board text added: "RX2"
- board text added: "SAT"
- board text added: "TX"
- board text added: "TX2"
- board text added: "URA"
- board text added: "VEN"

Commit message: gerbers
Routing:
- net +5V: track 139.4 -> 152.0 mm
- net GND: track 256.0 -> 262.2 mm
Other:
- board text added: "Art Controller V1"
- board text added: "Light-Up Planets"
